File: extension_v_1_1.sch (EAGLE design)
At the start: 5 parts

Commit message: Fixed bug where SDL and SDA pins were interchanged
Parts:
- R1, R2: value N.M. -> NOT MOUNTED
Connections:
- net VCC_3V3: no longer U$2POWER.IOREF
Changed lines of the file:
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@@
 <?xml version="1.0" encoding="utf-8"?>
 <!DOCTYPE eagle SYSTEM "eagle.dtd">
-<eagle version="6.4">
+<eagle version="7.2.0">
 <drawing>
 <settings>
@@
 <setting verticaltext="up"/>
 </settings>
-<grid distance="50" unitdist="mil" unit="mil" style="lines" multiple="1" display="yes" altdistance="0.01" altunitdist="inch" altunit="inch"/>
+<grid distance="0.05" unitdist="inch" unit="inch" style="lines" multiple="1" display="yes" altdistance="0.01" altunitdist="inch" altunit="inch"/>
 <layers>
 <layer number="1" name="Top" color="4" fill="1" visible="no" active="no"/>
@@
 <part name="U$2" library="ihpcb-arduino" deviceset="ARDUINO_UNO_SIZE_MCU_BOARD_NO_PWR" device=""/>
 <part name="PWR" library="ihpcb-pin_header" deviceset="M02X2" device=""/>
-<part name="R1" library="ihpcb-res_cap" deviceset="R0603" device="" value="N.M."/>
-<part name="R2" library="ihpcb-res_cap" deviceset="R0603" device="" value="N.M."/>
+<part name="R1" library="ihpcb-res_cap" deviceset="R0603" device="" value="NOT MOUNTED"/>
+<part name="R2" library="ihpcb-res_cap" deviceset="R0603" device="" value="NOT MOUNTED"/>
 </parts>
 <sheets>
@@
 </segment>
 <segment>
-<wire x1="55.88" y1="15.24" x2="55.88" y2="25.4" width="0.1524" layer="91"/>
-<junction x="55.88" y="25.4"/>
-<label x="55.88" y="25.4" size="1.778" layer="95" rot="R90"/>
-<pinref part="U$2" gate="POWER" pin="IOREF"/>
-</segment>
-<segment>
 <pinref part="PWR" gate="G$1" pin="4"/>
 <wire x1="-15.24" y1="60.96" x2="-7.62" y2="60.96" width="0.1524" layer="91"/>
@@
 <junction x="19.05" y="96.52"/>
 <label x="19.05" y="96.52" size="1.778" layer="95"/>
+<junction x="19.05" y="91.44"/>
 </segment>
 </net>
@@
 </sheet>
 </sheets>
+<errors>
+</errors>
 </schematic>
 </drawing>
